File: Board/RFID.brd (EAGLE design)
At the start: 160 x 100 mm, 24 parts, among them IC1 B82450A1084C000, Q8 125kHz, U1 HTRC11001T/02EE,11

Commit message: Placed board iter1
Parts:
- removed GPIO_5V, GPIO_POWER: 16V, led:LED5MM
- removed JP1, JP2: (no value), adafruit:1X20
- added C1: (no value), rcl:C0805
- added GLED, RLED: 16V, led:LED5MM
- added JP10: (no value), jumper:JP10Q
- added R1, R3, R5: (no value), adafruit:R0603
- added R2, R6, R9: 0ohm, adafruit:R0603
- JP3, JP4, JP5: device adafruit:1X20 -> jumper:JP10Q
- moved JP9 205.7 mm to (61.0, 26.7), turned to 268.2 degrees
- moved LS1 183.0 mm to (43.2, 24.1)
- moved JP8 179.6 mm to (12.7, 64.8), turned to 180 degrees
- moved R4 171.0 mm to (20.3, 19.1), turned to 180 degrees
- moved R7 171.0 mm to (25.4, 19.1), turned to 270 degrees
- moved JP6 169.7 mm to (61.0, 41.9)
- moved JP7 155.8 mm to (61.0, 17.8)
- moved C12 154.9 mm to (57.1, 35.6)
- moved C10 147.6 mm to (39.4, 35.6), turned to 180 degrees
- moved Q8 144.0 mm to (48.3, 35.6)
- moved C7 141.6 mm to (34.3, 48.3), turned to 180 degrees
- moved C6 140.6 mm to (34.3, 52.1), turned to 180 degrees
- moved JP3 111.5 mm to (49.5, 72.4), flipped to the bottom, turned to 180 degrees
- moved C4 109.8 mm to (30.5, 26.7)
- moved C5 109.8 mm to (30.5, 21.6)
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Connections:
- removed net PB3: JP4.16
- removed net PB4: JP4.14
- removed net PB5: JP4.15
- new net ANT3: C1.1, C3.1, R2.2, R3.2
- new net N$4: R1.1, R6.2
- new net N$5: JP4.1
- new net PA5: JP3.10
- new net PA6: JP3.8
- net 3V3: now also JP4.5; no longer JP1.8
- net 5V: now also JP4.3; no longer JP1.9
- net 5V_USB_CHG: now also JP3.13; no longer JP5.4
- net ADC1/10: now also JP5.3; no longer JP1.19
- net ADC1/11: now also JP5.5; no longer JP1.18
- net AGND: now also JP10.9; no longer JP5.16
- net ANT1: now also R5.2
- net ANT2: now also R1.2
- net AVDD: now also JP3.14; no longer JP4.4
- net BOOT0: now also JP4.14; no longer JP2.4
- net BUTTON1: now also JP5.18; no longer JP2.12
- net E5V: now also JP4.15; no longer JP1.3
- net ENTRY: now also JP5.6; no longer JP2.18
- net GND: now also GLED.K, JP3.1, JP3.12, JP4.13, JP4.2, JP5.19, RLED.K; no longer GPIO_5V.K, GPIO_POWER.K, JP1.10, JP1.11, JP1.4, JP2.10, JP4.5, JP5.10
- net I2C1_SDA: now also JP5.20; no longer JP2.11
- net IN: now also JP4.20; no longer JP2.1
- net IOREF: now also JP4.9; no longer JP1.6
- net N$2: now also GLED.A; no longer GPIO_POWER.A
- net N$3: now also RLED.A; no longer GPIO_5V.A
- net PA10: now also JP10.8; no longer JP4.17
- net PA11: now also JP3.7; no longer JP5.7
- net PA12: now also JP3.9; no longer JP5.6
- net PA8: now also JP10.18; no longer JP4.12
- net PA9: now also JP10.20; no longer JP4.11
- net PA_13: now also JP4.8; no longer JP2.7
- net PA_14: now also JP4.6; no longer JP2.8
- net PB1: now also JP10.17; no longer JP5.12
- net PB10: now also JP10.16; no longer JP4.13
- net PB11: now also JP3.3; no longer JP5.9
- net PB12: now also JP3.5; no longer JP5.8
- net PB13: now also JP10.11; no longer JP5.15
- net PB14: now also JP10.13; no longer JP5.14
- net PB15: now also JP10.15; no longer JP5.13
- net PB2: now also JP10.19; no longer JP5.11
- net PB6: now also JP3.4; no longer JP4.9
- net PB8: now also JP3.18; no longer JP4.2
- net PB9: now also JP3.16; no longer JP4.3
- net PC4: now also JP10.7; no longer JP5.17
- net PC4/PA2: now also JP10.6; no longer JP4.18
- net PC5: now also JP3.15; no longer JP5.3
- net PC5/PA3: now also JP10.4; no longer JP4.19
- net PC6: now also JP3.17; no longer JP5.2
- net PC7: now also JP3.2; no longer JP4.10
- net PC8: now also JP3.19; no longer JP5.1
- net PC9: now also JP3.20; no longer JP4.1
- net PC_11: now also JP4.19; no longer JP1.1
- net PC_12: now also JP4.18; no longer JP2.2
- net PC_14: now also JP5.16; no longer JP2.13
- net PC_15: now also JP5.14; no longer JP2.14
- net PD_2: now also JP4.17; no longer JP1.2
- net PF0: now also JP5.12; no longer JP2.15
- net PF1: now also JP5.10; no longer JP2.16
- net PWM2/1: now also JP4.4, JP5.13, LS1.2; no longer JP1.14, JP2.9
- net PWM2/2: now also JP5.11; no longer JP1.15
- net PWM3/3: now also JP5.7; no longer JP1.17
- net RESET: now also JP4.7; no longer JP1.7
- net RX: now also R6.1
- net SCLK: now also JP10.10; no longer JP4.6
- net SPI1_SSEL: now also JP5.9; no longer JP1.16
- net SPI_DIN: now also JP10.12, JP3.6; no longer JP4.8
- net SPI_DOUT: now also JP10.14; no longer JP4.7
- net TX1: now also C1.2, R3.1, R5.1, R9.1, R9.2
- net TX2: now also R2.1; no longer C3.1
- net VBAT: now also JP5.8; no longer JP2.17
- net VDD: now also JP4.16; no longer JP2.3
- net VIN: now also JP5.17; no longer JP1.12
- net ~ENTRY: now also JP5.4; no longer JP2.19, LS1.2
Routing:
- net 5V: track 0.00 -> 20.9 mm
- net N$2: track 0.00 -> 3.49 mm
- added copper zone on layer 1, net GND
Other:
- board size 160 x 100 mm -> 55.9 x 72.1 mm
- board text added: "Buzzer"
