File: Schematic/RFID.brd (EAGLE design)
At the start: 160 x 100 mm, 30 parts, among them IC1 B82450A1084C000, Q8 125kHz, U1 HTRC11001T/02EE,11

Commit message: Final routed board (Hopefully)
Parts:
- removed ENTRY, NOT_ENTRY: 16V, led:LED5MM
- removed IC1: B82450A1084C000, B82450A1084C000:B82450A_(11.4_X_3.5)
- removed JP2: (no value), adafruit:1X20
- removed R9: 0ohm, adafruit:R0603
- added GLED, RLED: 16V, led:LED5MM
- added JP10, JP3: (no value), jumper:JP10Q
- added R8: 0ohm, adafruit:R0603
- JP1: device adafruit:1X20 -> jumper:JP1
- JP4, JP5: device adafruit:1X20 -> jumper:JP10Q
- moved R5 255.4 mm to (53.8, 43.9)
- moved R1 250.3 mm to (53.3, 51.1)
- moved R3 248.1 mm to (45.2, 46.5), turned to 90 degrees
- moved R6 241.1 mm to (46.2, 50.8)
- moved R2 229.8 mm to (39.9, 47.8)
- moved C1 223.9 mm to (49.5, 46.5), turned to 270 degrees
- moved JP9 201.3 mm to (61.2, 20.8), turned to 90 degrees
- moved JP8 181.5 mm to (26.4, 62.0), turned to 180 degrees
- moved LS1 176.7 mm to (32.0, 23.4), turned to 180 degrees
- moved R7 172.0 mm to (9.40, 25.7), turned to 270 degrees
- moved R4 169.4 mm to (10.9, 20.8)
- moved JP6 159.6 mm to (61.2, 29.0)
- moved JP7 153.7 mm to (54.9, 20.1)
- moved C12 146.5 mm to (38.7, 37.8)
- moved C7 141.4 mm to (22.4, 54.9), turned to 90 degrees
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Connections:
- removed net ENTRY1: R3.2
- removed net PB3: JP4.16
- removed net PB4: JP4.14
- removed net PB5: JP4.15
- new net ANT4: C1.2, R3.1, R5.1, R8.2
- new net N$5: JP4.1
- new net PA15: JP4.4
- new net PA5: JP3.10
- new net PA6: JP3.8
- new net PA7: JP3.6
- net 3V3: now also JP4.5; no longer JP1.8
- net 5V: now also JP4.3, JP9.3; no longer JP1.9, JP9.2
- net 5V_USB_CHG: now also JP3.13; no longer JP5.4
- net ADC1/10: now also JP5.3; no longer JP1.19
- net ADC1/11: now also JP5.5; no longer JP1.18
- net AGND: now also JP10.9; no longer JP5.16
- net ANT1: now also JP1.1; no longer IC1.1
- net ANT2: now also JP1.2; no longer IC1.2
- net ANT3: now also R3.2
- net AVDD: now also JP3.14; no longer JP4.4
- net BOOT0: now also JP4.14; no longer JP2.4
- net BUTTON1: now also JP5.18; no longer JP2.12
- net E5V: now also JP4.15; no longer JP1.3
- net ENTRY: now also JP5.6; no longer JP2.18
- net GND: now also GLED.K, JP3.1, JP3.12, JP4.13, JP4.2, JP5.19, JP9.2, RLED.K; no longer ENTRY.K, JP1.10, JP1.11, JP1.4, JP2.10, JP4.5, JP5.10, JP9.3, NOT_ENTRY.K
- net I2C1_SDA: now also JP5.20; no longer JP2.11
- net IN: now also JP4.20; no longer JP2.1
- net IOREF: now also JP4.9; no longer JP1.6
- net N$2: now also GLED.A; no longer NOT_ENTRY.A
- net N$3: now also RLED.A; no longer ENTRY.A
- net PA10: now also JP10.8; no longer JP4.17
- net PA11: now also JP3.7; no longer JP5.7
- net PA12: now also JP3.9; no longer JP5.6
- net PA8: now also JP10.18; no longer JP4.12
- net PA9: now also JP10.20; no longer JP4.11
- net PA_13: now also JP4.8; no longer JP2.7
- net PA_14: now also JP4.6; no longer JP2.8
- net PB1: now also JP10.17; no longer JP5.12
- net PB10: now also JP10.16; no longer JP4.13
- net PB11: now also JP3.3; no longer JP5.9
- net PB12: now also JP3.5; no longer JP5.8
- net PB13: now also JP10.11; no longer JP5.15
- net PB14: now also JP10.13; no longer JP5.14
- net PB15: now also JP10.15; no longer JP5.13
- net PB2: now also JP10.19; no longer JP5.11
- net PB6: now also JP3.4; no longer JP4.9
- net PB8: now also JP3.18; no longer JP4.2
- net PB9: now also JP3.16; no longer JP4.3
- net PC4: now also JP10.7; no longer JP5.17
- net PC4/PA2: now also JP10.6; no longer JP4.18
- net PC5: now also JP3.15; no longer JP5.3
- net PC5/PA3: now also JP10.4; no longer JP4.19
- net PC6: now also JP3.17; no longer JP5.2
- net PC7: now also JP3.2; no longer JP4.10
- net PC8: now also JP3.19; no longer JP5.1
- net PC9: now also JP3.20; no longer JP4.1
- net PC_11: now also JP4.19; no longer JP1.1
- net PC_12: now also JP4.18; no longer JP2.2
- net PC_14: now also JP5.16; no longer JP2.13
- net PC_15: now also JP5.14; no longer JP2.14
- net PD_2: now also JP4.17; no longer JP1.2
- net PF0: now also JP5.12; no longer JP2.15
- net PF1: now also JP5.10; no longer JP2.16
- net PWM2/1: now also JP5.13; no longer JP1.14, JP2.9
- net PWM2/2: now also JP5.11; no longer JP1.15
- net PWM3/3: now also JP5.7; no longer JP1.17
- net RESET: now also JP4.7; no longer JP1.7
- net SCLK: now also JP10.10; no longer JP4.6
- net SPI1_SSEL: now also JP5.9; no longer JP1.16
- net SPI_DIN: now also JP10.12; no longer JP4.8
- net SPI_DOUT: now also JP10.14; no longer JP4.7
- net TX1: now also R8.1; no longer C1.2, R3.1, R5.1, R9.1, R9.2
- net VBAT: now also JP5.8; no longer JP2.17
- net VDD: now also JP4.16; no longer JP2.3
- net VIN: now also JP5.17; no longer JP1.12
- net ~ENTRY: now also JP5.4; no longer JP2.19
Routing:
- net 5V: track 0.00 -> 89.7 mm
- net SCLK: track 0.00 -> 28.0 mm
- net ENTRY: track 0.00 -> 26.9 mm
- net RX: track 0.00 -> 24.4 mm
- net SPI_DIN: track 0.00 -> 24.2 mm
- net SPI_DOUT: track 0.00 -> 23.7 mm
- net ~ENTRY: track 0.00 -> 19.0 mm
- net 3V3: track 0.00 -> 17.8 mm
- net TX2: track 0.00 -> 16.9 mm
- net TX1: track 0.00 -> 14.3 mm
- net CRY_N: track 0.00 -> 14.2 mm
- net ANT4: track 0.00 -> 14.2 mm
- net CRY_P: track 0.00 -> 14.1 mm
- net PWM2/1: track 0.00 -> 12.5 mm
- net ANT3: track 0.00 -> 12.3 mm
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- added copper zone on layer 1, net GND
Other:
- board size 160 x 100 mm -> 104.8 x 72.1 mm
- board text added: "Buzzer"
- board text added: "Impedance matching"
