File: Schematic/RFID.sch (EAGLE design)
At the start: 25 parts, among them IC1 B82450A1084C000, Q8 125kHz, U1 HTRC11001T/02EE,11

Commit message: Schematic v1
Parts:
- removed JP3: (no value), adafruit:PINHD-1X20
- added R1, R3, R5: (no value), adafruit:R-US_R0603
- added R2, R6, R9: 0ohm, adafruit:R-US_R0603
Connections:
- new net ANT3: C1.1, C3.1, R2.2
- new net ENTRY1: R3.2
- new net N$4: R1.1, R6.2
- net ANT1: now also R5.2
- net ANT2: now also R1.2
- net RX: now also R6.1
- net TX1: now also R3.1, R5.1, R9.1, R9.2
- net TX2: now also R2.1; no longer C1.1, C3.1
Changed lines of the file:
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@@
 <part name="JP1" library="adafruit" deviceset="PINHD-1X20" device=""/>
 <part name="JP2" library="adafruit" deviceset="PINHD-1X20" device=""/>
-<part name="JP3" library="adafruit" deviceset="PINHD-1X20" device=""/>
 <part name="JP4" library="adafruit" deviceset="PINHD-1X20" device=""/>
 <part name="JP5" library="adafruit" deviceset="PINHD-1X20" device=""/>
 <part name="IC1" library="B82450A1084C000" deviceset="B82450A1084C000" device=""/>
-<part name="R1" library="docu-dummy" library_urn="urn:adsk.eagle:library:215" deviceset="R" device=""/>
-<part name="R3" library="docu-dummy" library_urn="urn:adsk.eagle:library:215" deviceset="R" device=""/>
 <part name="C3" library="rcl" library_urn="urn:adsk.eagle:library:334" deviceset="C-US" device="C0805" package3d_urn="urn:adsk.eagle:package:23617/2"/>
 <part name="C4" library="rcl" library_urn="urn:adsk.eagle:library:334" deviceset="C-US" device="C0805" package3d_urn="urn:adsk.eagle:package:23617/2" value="10uF"/>
@@
 <part name="JP9" library="jumper" library_urn="urn:adsk.eagle:library:252" deviceset="JP2E" device="" package3d_urn="urn:adsk.eagle:package:15452/1"/>
 <part name="C1" library="rcl" library_urn="urn:adsk.eagle:library:334" deviceset="C-US" device="C0805" package3d_urn="urn:adsk.eagle:package:23617/2"/>
-<part name="R5" library="docu-dummy" library_urn="urn:adsk.eagle:library:215" deviceset="R" device=""/>
+<part name="R9" library="adafruit" deviceset="R-US_" device="R0603" value="0ohm"/>
+<part name="R2" library="adafruit" deviceset="R-US_" device="R0603" value="0ohm"/>
+<part name="R6" library="adafruit" deviceset="R-US_" device="R0603" value="0ohm"/>
+<part name="R1" library="adafruit" deviceset="R-US_" device="R0603"/>
+<part name="R3" library="adafruit" deviceset="R-US_" device="R0603"/>
+<part name="R5" library="adafruit" deviceset="R-US_" device="R0603"/>
 </parts>
 <sheets>
@@
 <attribute name="VALUE" x="92.71" y="154.94" size="1.778" layer="96"/>
 </instance>
-<instance part="JP3" gate="A" x="154.94" y="185.42" smashed="yes">
-<attribute name="NAME" x="148.59" y="211.455" size="1.778" layer="95"/>
-<attribute name="VALUE" x="148.59" y="154.94" size="1.778" layer="96"/>
-</instance>
 <instance part="JP4" gate="A" x="177.8" y="185.42" smashed="yes">
 <attribute name="NAME" x="171.45" y="211.455" size="1.778" layer="95"/>
@@
 <attribute name="VALUE" x="41.91" y="106.68" size="1.778" layer="96" align="center-left"/>
 </instance>
-<instance part="R1" gate="G$1" x="12.7" y="101.6" smashed="yes"/>
-<instance part="R3" gate="G$1" x="0" y="81.28" smashed="yes" rot="R180"/>
 <instance part="C3" gate="G$1" x="0" y="88.9" smashed="yes" rot="R90">
 <attribute name="NAME" x="-0.635" y="89.916" size="1.778" layer="95" rot="R90"/>
@@
 <attribute name="VALUE" x="-3.556" y="100.711" size="1.778" layer="96" rot="R180"/>
 </instance>
-<instance part="R5" gate="G$1" x="-7.62" y="96.52" smashed="yes" rot="R90"/>
+<instance part="R9" gate="G$1" x="-17.653" y="102.743" smashed="yes">
+<attribute name="NAME" x="-21.463" y="104.2416" size="1.778" layer="95"/>
+<attribute name="VALUE" x="-21.463" y="99.441" size="1.778" layer="96"/>
+</instance>
+<instance part="R2" gate="G$1" x="-17.653" y="90.043" smashed="yes">
+<attribute name="NAME" x="-21.463" y="91.5416" size="1.778" layer="95"/>
+<attribute name="VALUE" x="-21.463" y="86.741" size="1.778" layer="96"/>
+</instance>
+<instance part="R6" gate="G$1" x="-15.113" y="79.883" smashed="yes">
+<attribute name="NAME" x="-18.923" y="81.3816" size="1.778" layer="95"/>
+<attribute name="VALUE" x="-18.923" y="76.581" size="1.778" layer="96"/>
+</instance>
+<instance part="R1" gate="G$1" x="-2.413" y="79.883" smashed="yes">
+<attribute name="NAME" x="-6.223" y="81.3816" size="1.778" layer="95"/>
+<attribute name="VALUE" x="-6.223" y="76.581" size="1.778" layer="96"/>
+</instance>
+<instance part="R3" gate="G$1" x="-6.477" y="93.853" smashed="yes" rot="R270">
+<attribute name="NAME" x="-4.9784" y="97.663" size="1.778" layer="95" rot="R270"/>
+<attribute name="VALUE" x="-9.779" y="97.663" size="1.778" layer="96" rot="R270"/>
+</instance>
+<instance part="R5" gate="G$1" x="12.827" y="107.823" smashed="yes">
+<attribute name="NAME" x="9.017" y="109.3216" size="1.778" layer="95"/>
+<attribute name="VALUE" x="9.017" y="104.521" size="1.778" layer="96"/>
+</instance>
 </instances>
 <busses>
@@
 <pinref part="IC1" gate="G$1" pin="1"/>
 <wire x1="25.4" y1="101.6" x2="17.78" y2="101.6" width="0.1524" layer="91"/>
+<wire x1="17.78" y1="106.68" x2="17.78" y2="101.6" width="0.1524" layer="91"/>
+<pinref part="R5" gate="G$1" pin="2"/>
+<wire x1="17.907" y1="107.823" x2="17.907" y2="106.68" width="0.1524" layer="91"/>
+<wire x1="17.907" y1="106.68" x2="17.78" y2="106.68" width="0.1524" layer="91"/>
 </segment>
 </net>
@@
 <wire x1="5.08" y1="88.9" x2="5.08" y2="81.28" width="0.1524" layer="91"/>
 <junction x="5.08" y="88.9"/>
+<pinref part="R1" gate="G$1" pin="2"/>
+<wire x1="2.667" y1="79.883" x2="5.207" y2="81.28" width="0.1524" layer="91"/>
+<wire x1="5.207" y1="81.28" x2="5.08" y2="81.28" width="0.1524" layer="91"/>
 </segment>
 </net>
@@
 </segment>
 <segment>
-<pinref part="C3" gate="G$1" pin="1"/>
-<wire x1="-2.54" y1="88.9" x2="-7.62" y2="88.9" width="0.1524" layer="91"/>
-<label x="-15.24" y="88.9" size="1.778" layer="95" rot="R180" xref="yes"/>
-<pinref part="C1" gate="G$1" pin="1"/>
-<junction x="-2.54" y="88.9"/>
-<wire x1="-7.62" y1="88.9" x2="-15.24" y2="88.9" width="0.1524" layer="91"/>
-<wire x1="-2.54" y1="88.9" x2="-2.54" y2="93.98" width="0.1524" layer="91"/>
-<wire x1="-7.62" y1="91.44" x2="-7.62" y2="88.9" width="0.1524" layer="91"/>
-<junction x="-7.62" y="88.9"/>
+<label x="-25.4" y="88.9" size="1.778" layer="95" rot="R180" xref="yes"/>
+<pinref part="R2" gate="G$1" pin="1"/>
+<wire x1="-27.94" y1="88.9" x2="-22.733" y2="88.9" width="0.1524" layer="91"/>
+<wire x1="-22.733" y1="88.9" x2="-22.733" y2="90.043" width="0.1524" layer="91"/>
 </segment>
 </net>
@@
 </segment>
 <segment>
+<wire x1="-2.54" y1="101.6" x2="-6.477" y2="101.6" width="0.1524" layer="91"/>
+<wire x1="-6.477" y1="101.6" x2="-12.7" y2="101.6" width="0.1524" layer="91"/>
 <wire x1="7.62" y1="101.6" x2="-2.54" y2="101.6" width="0.1524" layer="91"/>
-<label x="-15.24" y="101.6" size="1.778" layer="95" rot="R180" xref="yes"/>
 <pinref part="C1" gate="G$1" pin="2"/>
-<wire x1="-2.54" y1="101.6" x2="-15.24" y2="101.6" width="0.1524" layer="91"/>
-<junction x="-2.54" y="101.6"/>
+<wire x1="7.62" y1="107.823" x2="7.62" y2="101.6" width="0.1524" layer="91"/>
+<pinref part="R9" gate="G$1" pin="2"/>
+<wire x1="-12.573" y1="102.743" x2="-12.7" y2="102.743" width="0.1524" layer="91"/>
+<wire x1="-12.7" y1="102.743" x2="-12.7" y2="101.6" width="0.1524" layer="91"/>
+<pinref part="R3" gate="G$1" pin="1"/>
+<wire x1="-6.477" y1="98.933" x2="-6.477" y2="101.6" width="0.1524" layer="91"/>
+<pinref part="R5" gate="G$1" pin="1"/>
+<wire x1="7.62" y1="107.823" x2="7.747" y2="107.823" width="0.1524" layer="91"/>
+</segment>
+<segment>
+<wire x1="-22.86" y1="101.6" x2="-25.4" y2="101.6" width="0.1524" layer="91"/>
+<label x="-25.4" y="101.6" size="1.778" layer="95" rot="R180" xref="yes"/>
+<pinref part="R9" gate="G$1" pin="1"/>
+<wire x1="-22.733" y1="102.743" x2="-22.86" y2="102.743" width="0.1524" layer="91"/>
+<wire x1="-22.86" y1="102.743" x2="-22.86" y2="101.6" width="0.1524" layer="91"/>
 </segment>
 </net>
@@
 </segment>
 <segment>
-<wire x1="-5.08" y1="81.28" x2="-17.78" y2="81.28" width="0.1524" layer="91"/>
-<label x="-17.78" y="81.28" size="1.778" layer="95" rot="R180" xref="yes"/>
+<wire x1="-25.4" y1="78.74" x2="-27.94" y2="78.74" width="0.1524" layer="91"/>
+<label x="-27.94" y="78.74" size="1.778" layer="95" rot="R180" xref="yes"/>
+<label x="-27.94" y="78.74" size="1.778" layer="95" rot="R180" xref="yes"/>
+<pinref part="R6" gate="G$1" pin="1"/>
+<wire x1="-20.193" y1="79.883" x2="-25.4" y2="79.883" width="0.1524" layer="91"/>
+<wire x1="-25.4" y1="79.883" x2="-25.4" y2="78.74" width="0.1524" layer="91"/>
 </segment>
 </net>
@@
 </segment>
 </net>
+<net name="ANT3" class="0">
+<segment>
+<pinref part="C3" gate="G$1" pin="1"/>
+<wire x1="-2.54" y1="88.9" x2="-12.573" y2="88.9" width="0.1524" layer="91"/>
+<pinref part="C1" gate="G$1" pin="1"/>
+<junction x="-2.54" y="88.9"/>
+<wire x1="-2.54" y1="88.9" x2="-2.54" y2="93.98" width="0.1524" layer="91"/>
+<pinref part="R2" gate="G$1" pin="2"/>
+<wire x1="-12.573" y1="90.043" x2="-12.573" y2="88.9" width="0.1524" layer="91"/>
+</segment>
+</net>
+<net name="N$4" class="0">
+<segment>
+<pinref part="R6" gate="G$1" pin="2"/>
+<pinref part="R1" gate="G$1" pin="1"/>
+<wire x1="-10.033" y1="79.883" x2="-7.493" y2="79.883" width="0.1524" layer="91"/>
+</segment>
+</net>
+<net name="ENTRY1" class="0">
+<segment>
+<pinref part="R3" gate="G$1" pin="2"/>
+<wire x1="-6.477" y1="88.773" x2="-6.477" y2="88.9" width="0.1524" layer="91"/>
+</segment>
+</net>

Commit message: Placed board iter1
Parts:
- renumbered GPIO_5V to ENTRY, GPIO_POWER to NOT_ENTRY
Changed lines of the file:
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@@
 <part name="R7" library="adafruit" deviceset="R-US_" device="R0603" value="0.2k"/>
 <part name="R4" library="adafruit" deviceset="R-US_" device="R0603" value="0.2k"/>
-<part name="GPIO_POWER" library="led" library_urn="urn:adsk.eagle:library:259" deviceset="LED" device="5MM" package3d_urn="urn:adsk.eagle:package:15799/2" value="16V"/>
-<part name="GPIO_5V" library="led" library_urn="urn:adsk.eagle:library:259" deviceset="LED" device="5MM" package3d_urn="urn:adsk.eagle:package:15799/2" value="16V"/>
+<part name="NOT_ENTRY" library="led" library_urn="urn:adsk.eagle:library:259" deviceset="LED" device="5MM" package3d_urn="urn:adsk.eagle:package:15799/2" value="16V"/>
+<part name="ENTRY" library="led" library_urn="urn:adsk.eagle:library:259" deviceset="LED" device="5MM" package3d_urn="urn:adsk.eagle:package:15799/2" value="16V"/>
 <part name="LS1" library="PS1240P02BT" deviceset="PS1240P02BT" device=""/>
 <part name="JP9" library="jumper" library_urn="urn:adsk.eagle:library:252" deviceset="JP2E" device="" package3d_urn="urn:adsk.eagle:package:15452/1"/>
@@
 <attribute name="VALUE" x="191.643" y="114.173" size="1.778" layer="96" rot="R90"/>
 </instance>
-<instance part="GPIO_POWER" gate="G$1" x="188.722" y="127.762" smashed="yes" rot="R180">
+<instance part="NOT_ENTRY" gate="G$1" x="188.722" y="127.762" smashed="yes" rot="R180">
 <attribute name="VALUE" x="193.421" y="131.064" size="1.778" layer="96" rot="R270"/>
 </instance>
-<instance part="GPIO_5V" gate="G$1" x="178.562" y="128.778" smashed="yes" rot="R180">
+<instance part="ENTRY" gate="G$1" x="178.562" y="128.778" smashed="yes" rot="R180">
 <attribute name="VALUE" x="183.261" y="132.08" size="1.778" layer="96" rot="R270"/>
 </instance>
@@
 <segment>
 <label x="178.562" y="136.398" size="1.778" layer="95" rot="R90" xref="yes"/>
-<pinref part="GPIO_5V" gate="G$1" pin="C"/>
+<pinref part="ENTRY" gate="G$1" pin="C"/>
 <wire x1="178.562" y1="133.858" x2="178.562" y2="136.398" width="0.1524" layer="91"/>
 </segment>
 <segment>
 <label x="188.722" y="136.398" size="1.778" layer="95" rot="R90" xref="yes"/>
-<pinref part="GPIO_POWER" gate="G$1" pin="C"/>
+<pinref part="NOT_ENTRY" gate="G$1" pin="C"/>
 <wire x1="188.722" y1="132.842" x2="188.722" y2="136.398" width="0.1524" layer="91"/>
 </segment>
@@
 <net name="N$3" class="0">
 <segment>
-<pinref part="GPIO_5V" gate="G$1" pin="A"/>
+<pinref part="ENTRY" gate="G$1" pin="A"/>
 <pinref part="R7" gate="G$1" pin="1"/>
 <wire x1="178.562" y1="126.238" x2="178.562" y2="121.793" width="0.1524" layer="91"/>
@@
 <net name="N$2" class="0">
 <segment>
-<pinref part="GPIO_POWER" gate="G$1" pin="A"/>
+<pinref part="NOT_ENTRY" gate="G$1" pin="A"/>
 <pinref part="R4" gate="G$1" pin="2"/>
 <wire x1="188.722" y1="125.222" x2="188.341" y2="125.222" width="0.1524" layer="91"/>

Commit message: Final routed board (Hopefully)
Parts:
- removed IC1: B82450A1084C000, B82450A1084C000:B82450A1084C000
- removed JP2: (no value), adafruit:PINHD-1X20
- added JP10, JP3: (no value), jumper:JP10Q
- JP1: device adafruit:PINHD-1X20 -> jumper:JP1E
- JP4, JP5: device adafruit:PINHD-1X20 -> jumper:JP10Q
- renumbered ENTRY to RLED, NOT_ENTRY to GLED, R9 to R8
Connections:
- removed net ENTRY1: R3.2
- removed net PB3: JP4.16
- removed net PB4: JP4.14
- removed net PB5: JP4.15
- new net ANT4: C1.2, R3.1, R5.1, R8.2
- new net N$5: JP4.1
- new net PA15: JP4.4
- new net PA5: JP3.10
- new net PA6: JP3.8
- new net PA7: JP3.6
- net 3V3: now also JP4.5; no longer JP1.8
- net 5V: now also JP4.3, JP9.3; no longer JP1.9, JP9.2
- net 5V_USB_CHG: now also JP3.13; no longer JP5.4
- net ADC1/10: now also JP5.3; no longer JP1.19
- net ADC1/11: now also JP5.5; no longer JP1.18
- net AGND: now also JP10.9; no longer JP5.16
- net ANT1: now also JP1.1; no longer IC1.1
- net ANT2: now also JP1.2; no longer IC1.2
- net ANT3: now also R3.2
- net AVDD: now also JP3.14; no longer JP4.4
- net BOOT0: now also JP4.14; no longer JP2.4
- net BUTTON1: now also JP5.18; no longer JP2.12
- net E5V: now also JP4.15; no longer JP1.3
- net ENTRY: now also JP5.6; no longer JP2.18
- net GND: now also JP3.1, JP3.12, JP4.13, JP4.2, JP5.19, JP9.2; no longer JP1.10, JP1.11, JP1.4, JP2.10, JP4.5, JP5.10, JP9.3
- net I2C1_SDA: now also JP5.20; no longer JP2.11
- net IN: now also JP4.20; no longer JP2.1
- net IOREF: now also JP4.9; no longer JP1.6
- net PA10: now also JP10.8; no longer JP4.17
- net PA11: now also JP3.7; no longer JP5.7
- net PA12: now also JP3.9; no longer JP5.6
- net PA8: now also JP10.18; no longer JP4.12
- net PA9: now also JP10.20; no longer JP4.11
- net PA_13: now also JP4.8; no longer JP2.7
- net PA_14: now also JP4.6; no longer JP2.8
- net PB1: now also JP10.17; no longer JP5.12
- net PB10: now also JP10.16; no longer JP4.13
- net PB11: now also JP3.3; no longer JP5.9
- net PB12: now also JP3.5; no longer JP5.8
- net PB13: now also JP10.11; no longer JP5.15
- net PB14: now also JP10.13; no longer JP5.14
- net PB15: now also JP10.15; no longer JP5.13
- net PB2: now also JP10.19; no longer JP5.11
- net PB6: now also JP3.4; no longer JP4.9
- net PB8: now also JP3.18; no longer JP4.2
- net PB9: now also JP3.16; no longer JP4.3
- net PC4: now also JP10.7; no longer JP5.17
- net PC4/PA2: now also JP10.6; no longer JP4.18
- net PC5: now also JP3.15; no longer JP5.3
- net PC5/PA3: now also JP10.4; no longer JP4.19
- net PC6: now also JP3.17; no longer JP5.2
- net PC7: now also JP3.2; no longer JP4.10
- net PC8: now also JP3.19; no longer JP5.1
- net PC9: now also JP3.20; no longer JP4.1
- net PC_11: now also JP4.19; no longer JP1.1
- net PC_12: now also JP4.18; no longer JP2.2
- net PC_14: now also JP5.16; no longer JP2.13
- net PC_15: now also JP5.14; no longer JP2.14
- net PD_2: now also JP4.17; no longer JP1.2
- net PF0: now also JP5.12; no longer JP2.15
- net PF1: now also JP5.10; no longer JP2.16
- net PWM2/1: now also JP5.13; no longer JP1.14, JP2.9
- net PWM2/2: now also JP5.11; no longer JP1.15
- net PWM3/3: now also JP5.7; no longer JP1.17
- net RESET: now also JP4.7; no longer JP1.7
- net SCLK: now also JP10.10; no longer JP4.6
- net SPI1_SSEL: now also JP5.9; no longer JP1.16
- net SPI_DIN: now also JP10.12; no longer JP4.8
- net SPI_DOUT: now also JP10.14; no longer JP4.7
- net TX1: no longer C1.2, R3.1, R5.1, R8.2
- net VBAT: now also JP5.8; no longer JP2.17
- net VDD: now also JP4.16; no longer JP2.3
- net VIN: now also JP5.17; no longer JP1.12
- net ~ENTRY: now also JP5.4; no longer JP2.19
Other:
- moved on the sheet: R3
